Commit message: Update turtlebot3_gazebo

File: ros_ws/src/turtlebot3_gazebo/urdf/turtlebot3_burger_cam1.urdf (robot description, URDF)
Before this commit: robot turtlebot3_burger_cam, 11 links, 10 joints
Links:
- added link robot1/camera_depth_frame
Joints:
- added joint robot1/camera_depth_optical_joint: type fixed, parent robot1/camera_depth_frame, child robot1/camera_depth_optical_frame, origin xyz=0 0 0 rpy=-1.5707 0 -1.57
- joint robot1/camera_depth_joint: child robot1/camera_depth_optical_frame -> robot1/camera_depth_frame; origin xyz=0 0 0 rpy=0 0 0 -> xyz=0.003 0.000 0.009 rpy=0 0 0

File: ros_ws/src/turtlebot3_gazebo/urdf/turtlebot3_burger_cam2.urdf (robot description, URDF)
Before this commit: robot turtlebot3_burger_cam, 11 links, 10 joints
Links:
- added link robot2/camera_depth_frame
Joints:
- added joint robot2/camera_depth_optical_joint: type fixed, parent robot2/camera_depth_frame, child robot2/camera_depth_optical_frame, origin xyz=0 0 0 rpy=-1.5707 0 -1.57
- joint robot2/camera_depth_joint: child robot2/camera_depth_optical_frame -> robot2/camera_depth_frame
